Commit message: add control pkg

File: src/vx300s_description/urdf/vx300s.urdf.xacro (robot description, xacro)
@@ -6,4 +6,11 @@
   <!-- use_world_frame -->
 <xacro:macro name="vx300s">
+<link name="world"/>
+    <joint name="fixed" type="fixed">
+      <parent
+        link="world"/>
+      <child
+        link="vx300s/base_link"/>
+    </joint>
  <link name="vx300s/base_link">
      <visual>
