Commit message: simulation works but some few error, which is annoy but can ignore anyway...

File: src/vx300s_description/urdf/vx300s.urdf (robot description, URDF)
Before this commit: robot vx300s, 14 links, 13 joints
Links:
- link vx300s/shoulder_link: geometry collision mesh filename=package://vx300s_description/vx300s_meshes/shoulder.stl scale=0.001 0.001 0.001; visual mesh filename=package://vx300s_description/vx300s_meshes/shoulder.stl scale=0.001 0.001 0.001

File: src/vx300s_description/urdf/vx300s.xacro (robot description, xacro)
@@ -2,13 +2,13 @@
 <robot xmlns:xacro="http://www.ros.org/wiki/xacro" name="vx300s">
   <material name="interbotix_black">
-    <texture filename="package://vx300s_description/vx300s_meshes/interbotix_black.png"/>
+    <texture filename="file:///home/yc/vx300s-single-sim/src/vx300s_description/vx300s_meshes/interbotix_black.png"/>
   </material>
   <!-- use_world_frame -->
-<xacro:macro name="base_link">
+<xacro:macro name="vx300s">
  <link name="vx300s/base_link">
      <visual>
        <origin rpy="0 0 1.5707963267948966" xyz="0 0 0"/>
        <geometry>
-         <mesh filename="package://vx300s_description/vx300s_meshes/base.stl" scale="0.001 0.001 0.001"/>
+         <mesh filename="file:///home/yc/vx300s-single-sim/src/vx300s_description/vx300s_meshes/base.stl" scale="0.001 0.001 0.001"/>
        </geometry>
        <material name="interbotix_black"/>
@@ -17,5 +17,5 @@
        <origin rpy="0 0 1.5707963267948966" xyz="0 0 0"/>
        <geometry>
-         <mesh filename="package://vx300s_description/vx300s_meshes/base.stl" scale="0.001 0.001 0.001"/>
+         <mesh filename="file:///home/yc/vx300s-single-sim/src/vx300s_description/vx300s_meshes/base.stl" scale="0.001 0.001 0.001"/>
        </geometry>
      </collision>
@@ -34,11 +34,9 @@
     <dynamics damping="0.1" friction="0.1"/>
  </joint>
-</xacro:macro>
-<xacro:macro name="shoulder_link">
   <link name="vx300s/shoulder_link">
     <visual>
       <origin rpy="0 0 1.5707963267948966" xyz="0 0 -0.003"/>
       <geometry>
-        <mesh filename="package://vx300s_description/vx300s_meshes/shoulder.stl" scale="0.001 0.001 0.001"/>
+        <mesh filename="file:///home/yc/vx300s-single-sim/src/vx300s_description/vx300s_meshes/shoulder.stl" scale="0.001 0.001 0.001"/>
       </geometry>
       <material name="interbotix_black"/>
@@ -47,5 +45,5 @@
       <origin rpy="0 0 1.5707963267948966" xyz="0 0 -0.003"/>
       <geometry>
-        <mesh filename="package://vx300s_description/vx300s_meshes/shoulder.stl" scale="0.001 0.001 0.001"/>
+        <mesh filename="file:///home/yc/vx300s-single-sim/src/vx300s_description/vx300s_meshes/shoulder.stl" scale="0.001 0.001 0.001"/>
       </geometry>
     </collision>
@@ -64,11 +62,9 @@
     <dynamics damping="0.1" friction="0.1"/>
   </joint>
-</xacro:macro>
-<xacro:macro name="upper_arm_link">
   <link name="vx300s/upper_arm_link">
     <visual>
       <origin rpy="0 0 1.5707963267948966" xyz="0 0 0"/>
       <geometry>
-        <mesh filename="package://vx300s_description/vx300s_meshes/upper_arm.stl" scale="0.001 0.001 0.001"/>
+        <mesh filename="file:///home/yc/vx300s-single-sim/src/vx300s_description/vx300s_meshes/upper_arm.stl" scale="0.001 0.001 0.001"/>
       </geometry>
       <material name="interbotix_black"/>
@@ -77,5 +73,5 @@
       <origin rpy="0 0 1.5707963267948966" xyz="0 0 0"/>
       <geometry>
-        <mesh filename="package://vx300s_description/vx300s_meshes/upper_arm.stl" scale="0.001 0.001 0.001"/>
+        <mesh filename="file:///home/yc/vx300s-single-sim/src/vx300s_description/vx300s_meshes/upper_arm.stl" scale="0.001 0.001 0.001"/>
       </geometry>
     </collision>
@@ -94,11 +90,9 @@
     <dynamics damping="0.1" friction="0.1"/>
   </joint>
-</xacro:macro>
-<xacro:macro name="upper_forearm_link">
   <link name="vx300s/upper_forearm_link">
     <visual>
       <origin rpy="0 0 0" xyz="0 0 0"/>
       <geometry>
-        <mesh filename="package://vx300s_description/vx300s_meshes/upper_forearm.stl" scale="0.001 0.001 0.001"/>
+        <mesh filename="file:///home/yc/vx300s-single-sim/src/vx300s_description/vx300s_meshes/upper_forearm.stl" scale="0.001 0.001 0.001"/>
       </geometry>
       <material name="interbotix_black"/>
@@ -107,5 +101,5 @@
       <origin rpy="0 0 0" xyz="0 0 0"/>
       <geometry>
-        <mesh filename="package://vx300s_description/vx300s_meshes/upper_forearm.stl" scale="0.001 0.001 0.001"/>
+        <mesh filename="file:///home/yc/vx300s-single-sim/src/vx300s_description/vx300s_meshes/upper_forearm.stl" scale="0.001 0.001 0.001"/>
       </geometry>
     </collision>
@@ -124,11 +118,9 @@
     <dynamics damping="0.1" friction="0.1"/>
   </joint>
-</xacro:macro>
-<xacro:macro name="lower_forearm_link">
   <link name="vx300s/lower_forearm_link">
     <visual>
       <origin rpy="3.141592653589793 0 0" xyz="0 0 0"/>
       <geometry>
-        <mesh filename="package://vx300s_description/vx300s_meshes/lower_forearm.stl" scale="0.001 0.001 0.001"/>
+        <mesh filename="file:///home/yc/vx300s-single-sim/src/vx300s_description/vx300s_meshes/lower_forearm.stl" scale="0.001 0.001 0.001"/>
       </geometry>
       <material name="interbotix_black"/>
@@ -137,5 +129,5 @@
       <origin rpy="3.141592653589793 0 0" xyz="0 0 0"/>
       <geometry>
-        <mesh filename="package://vx300s_description/vx300s_meshes/lower_forearm.stl" scale="0.001 0.001 0.001"/>
+        <mesh filename="file:///home/yc/vx300s-single-sim/src/vx300s_description/vx300s_meshes/lower_forearm.stl" scale="0.001 0.001 0.001"/>
       </geometry>
     </collision>
@@ -154,11 +146,9 @@
     <dynamics damping="0.1" friction="0.1"/>
   </joint>
-</xacro:macro>
-<xacro:macro name="wrist_link">
   <link name="vx300s/wrist_link">
     <visual>
       <origin rpy="0 0 1.5707963267948966" xyz="0 0 0"/>
       <geometry>
-        <mesh filename="package://vx300s_description/vx300s_meshes/wrist.stl" scale="0.001 0.001 0.001"/>
+        <mesh filename="file:///home/yc/vx300s-single-sim/src/vx300s_description/vx300s_meshes/wrist.stl" scale="0.001 0.001 0.001"/>
       </geometry>
       <material name="interbotix_black"/>
@@ -167,5 +157,5 @@
       <origin rpy="0 0 1.5707963267948966" xyz="0 0 0"/>
       <geometry>
-        <mesh filename="package://vx300s_description/vx300s_meshes/wrist.stl" scale="0.001 0.001 0.001"/>
+        <mesh filename="file:///home/yc/vx300s-single-sim/src/vx300s_description/vx300s_meshes/wrist.stl" scale="0.001 0.001 0.001"/>
       </geometry>
     </collision>
@@ -185,11 +175,9 @@
     <dynamics damping="0.1" friction="0.1"/>
   </joint>
-</xacro:macro>
-<xacro:macro name="gripper_link">
   <link name="vx300s/gripper_link">
     <visual>
       <origin rpy="0 0 1.5707963267948966" xyz="-0.02 0 0"/>
       <geometry>
-        <mesh filename="package://vx300s_description/vx300s_meshes/gripper.stl" scale="0.001 0.001 0.001"/>
+        <mesh filename="file:///home/yc/vx300s-single-sim/src/vx300s_description/vx300s_meshes/gripper.stl" scale="0.001 0.001 0.001"/>
       </geometry>
       <material name="interbotix_black"/>
@@ -198,5 +186,5 @@
       <origin rpy="0 0 1.5707963267948966" xyz="-0.02 0 0"/>
       <geometry>
-        <mesh filename="package://vx300s_description/vx300s_meshes/gripper.stl" scale="0.001 0.001 0.001"/>
+        <mesh filename="file:///home/yc/vx300s-single-sim/src/vx300s_description/vx300s_meshes/gripper.stl" scale="0.001 0.001 0.001"/>
       </geometry>
     </collision>
@@ -213,6 +201,4 @@
     <child link="vx300s/ee_arm_link"/>
   </joint>
-</xacro:macro>
-<xacro:macro name="ee_arm_link">
   <link name="vx300s/ee_arm_link">
     <inertial>
@@ -229,11 +215,9 @@
     <dynamics damping="0.1" friction="0.1"/>
   </joint>
-</xacro:macro>
-<xacro:macro name="gripper_prop_link">
  <link name="vx300s/gripper_prop_link">
     <visual>
       <origin rpy="0 0 1.5707963267948966" xyz="-0.0685 0 0"/>
       <geometry>
-        <mesh filename="package://vx300s_description/vx300s_meshes/gripper_prop.stl" scale="0.001 0.001 0.001"/>
+        <mesh filename="file:///home/yc/vx300s-single-sim/src/vx300s_description/vx300s_meshes/gripper_prop.stl" scale="0.001 0.001 0.001"/>
       </geometry>
       <material name="interbotix_black"/>
@@ -242,5 +226,5 @@
       <origin rpy="0 0 1.5707963267948966" xyz="-0.0685 0 0"/>
       <geometry>
-        <mesh filename="package://vx300s_description/vx300s_meshes/gripper_prop.stl" scale="0.001 0.001 0.001"/>
+        <mesh filename="file:///home/yc/vx300s-single-sim/src/vx300s_description/vx300s_meshes/gripper_prop.stl" scale="0.001 0.001 0.001"/>
       </geometry>
     </collision>
@@ -251,14 +235,12 @@
     </inertial>
   </link>
-</xacro:macro>
   <!-- If the AR tag is being used, then add the AR tag mount -->
   <!-- show_ar_tag -->
   <!-- If the gripper bar is being used, then also add the gripper bar -->
-<xacro:macro name="gripper_bar_link">
   <link name="vx300s/gripper_bar_link">
     <visual>
       <origin rpy="0 0 1.5707963267948966" xyz="-0.063 0 0"/>
       <geometry>
-        <mesh filename="package://vx300s_description/vx300s_meshes/gripper_bar.stl" scale="0.001 0.001 0.001"/>
+        <mesh filename="file:///home/yc/vx300s-single-sim/src/vx300s_description/vx300s_meshes/gripper_bar.stl" scale="0.001 0.001 0.001"/>
       </geometry>
       <material name="interbotix_black"/>
@@ -267,5 +249,5 @@
       <origin rpy="0 0 1.5707963267948966" xyz="-0.063 0 0"/>
       <geometry>
-        <mesh filename="package://vx300s_description/vx300s_meshes/gripper_bar.stl" scale="0.001 0.001 0.001"/>
+        <mesh filename="file:///home/yc/vx300s-single-sim/src/vx300s_description/vx300s_meshes/gripper_bar.stl" scale="0.001 0.001 0.001"/>
       </geometry>
     </collision>
@@ -282,6 +264,4 @@
     <child link="vx300s/gripper_bar_link"/>
   </joint>
-</xacro:macro>
-<xacro:macro name="fingers_link">
 <joint name="ee_bar" type="fixed">
     <axis xyz="1 0 0"/>
@@ -296,12 +276,9 @@
     </inertial>
   </link>
-</xacro:macro>
-  <!-- If the gripper fingers are being used, add those as well -->
-<xacro:macro name="left_finger_link">
   <link name="vx300s/left_finger_link">
     <visual>
       <origin rpy="1.5707963267948966 -3.141592653589793 1.5707963267948966" xyz="-0.0404 -0.0575 0"/>
       <geometry>
-        <mesh filename="package://vx300s_description/vx300s_meshes/gripper_finger.stl" scale="0.001 0.001 0.001"/>
+        <mesh filename="file:///home/yc/vx300s-single-sim/src/vx300s_description/vx300s_meshes/gripper_finger.stl" scale="0.001 0.001 0.001"/>
       </geometry>
       <material name="interbotix_black"/>
@@ -310,5 +287,5 @@
       <origin rpy="1.5707963267948966 -3.141592653589793 1.5707963267948966" xyz="-0.0404 -0.0575 0"/>
       <geometry>
-        <mesh filename="package://vx300s_description/vx300s_meshes/gripper_finger.stl" scale="0.001 0.001 0.001"/>
+        <mesh filename="file:///home/yc/vx300s-single-sim/src/vx300s_description/vx300s_meshes/gripper_finger.stl" scale="0.001 0.001 0.001"/>
       </geometry>
     </collision>
@@ -327,6 +304,4 @@
     <dynamics damping="0.1" friction="0.1"/>
   </joint>
-</xacro:macro>
-<xacro:macro name="right_finger_link">
 <joint name="right_finger" type="prismatic">
     <axis xyz="0 1 0"/>
@@ -342,5 +317,5 @@
       <origin rpy="-1.5707963267948966 3.141592653589793 -1.5707963267948966" xyz="-0.0404 0.0575 0 "/>
       <geometry>
-        <mesh filename="package://vx300s_description/vx300s_meshes/gripper_finger.stl" scale="0.001 0.001 0.001"/>
+        <mesh filename="file:///home/yc/vx300s-single-sim/src/vx300s_description/vx300s_meshes/gripper_finger.stl" scale="0.001 0.001 0.001"/>
       </geometry>
       <material name="interbotix_black"/>
@@ -349,5 +324,5 @@
       <origin rpy="-1.5707963267948966 3.141592653589793 -1.5707963267948966" xyz="-0.0404 0.0575 0 "/>
       <geometry>
-        <mesh filename="package://vx300s_description/vx300s_meshes/gripper_finger.stl" scale="0.001 0.001 0.001"/>
+        <mesh filename="file:///home/yc/vx300s-single-sim/src/vx300s_description/vx300s_meshes/gripper_finger.stl" scale="0.001 0.001 0.001"/>
       </geometry>
     </collision>
@@ -358,6 +333,4 @@
     </inertial>
   </link>
-</xacro:macro>
-<xacro:macro name="ee_gripper_link">
 <joint name="ee_gripper" type="fixed">
     <axis xyz="1 0 0"/>
@@ -373,20 +346,4 @@
   </link>
 </xacro:macro>
-    <xacro:base_link/>
-    <xacro:shoulder_link/>
-    <xacro:upper_arm_link/>
-    <xacro:upper_forearm_link/>
-    <xacro:lower_forearm_link/>
-    <xacro:wrist_link/>
-    <xacro:gripper_link/>
-    <xacro:ee_arm_link/>
-    <xacro:gripper_prop_link/>
-    <xacro:gripper_bar_link/>
-    <xacro:fingers_link/>
-    <xacro:left_finger_link/>
-    <xacro:right_finger_link/>
-    <xacro:ee_gripper_link/>
-  <!-- show_gripper_fingers -->
-  <!-- show_gripper_bar -->
-  <!-- use_gripper -->
+    <xacro:vx300s/>
 </robot>

Commit message: pinocchio is good

File: src/vx300s_description/urdf/vx300s.urdf (robot description, URDF)
Before this commit: robot vx300s, 14 links, 13 joints
Links:
- link vx300s/base_link: geometry collision mesh filename=/home/yc/vx300s-single-sim/src/vx300s_description/vx300s_me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 scale=0.001 0.001 0.001; visual mesh filename=/home/yc/vx300s-single-sim/src/vx300s_description/vx300s_me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 scale=0.001 0.001 0.001
- link vx300s/gripper_bar_link: geometry collision mesh filename=/home/yc/vx300s-single-sim/src/vx300s_description/vx300s_me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 scale=0.001 0.001 0.001; visual mesh filename=/home/yc/vx300s-single-sim/src/vx300s_description/vx300s_me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 scale=0.001 0.001 0.001
- link vx300s/gripper_link: geometry collision mesh filename=/home/yc/vx300s-single-sim/src/vx300s_description/vx300s_me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 scale=0.001 0.001 0.001; visual mesh filename=/home/yc/vx300s-single-sim/src/vx300s_description/vx300s_me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 scale=0.001 0.001 0.001
- link vx300s/gripper_prop_link: geometry collision mesh filename=/home/yc/vx300s-single-sim/src/vx300s_description/vx300s_me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 scale=0.001 0.001 0.001; visual mesh filename=/home/yc/vx300s-single-sim/src/vx300s_description/vx300s_me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 scale=0.001 0.001 0.001
- link vx300s/left_finger_link: geometry collision mesh filename=/home/yc/vx300s-single-sim/src/vx300s_description/vx300s_me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 scale=0.001 0.001 0.001; visual mesh filename=/home/yc/vx300s-single-sim/src/vx300s_description/vx300s_me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 scale=0.001 0.001 0.001
- link vx300s/lower_forearm_link: geometry collision mesh filename=/home/yc/vx300s-single-sim/src/vx300s_description/vx300s_me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 scale=0.001 0.001 0.001; visual mesh filename=/home/yc/vx300s-single-sim/src/vx300s_description/vx300s_me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 scale=0.001 0.001 0.001
- link vx300s/right_finger_link: geometry collision mesh filename=/home/yc/vx300s-single-sim/src/vx300s_description/vx300s_me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 scale=0.001 0.001 0.001; visual mesh filename=/home/yc/vx300s-single-sim/src/vx300s_description/vx300s_me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 scale=0.001 0.001 0.001
- link vx300s/shoulder_link: geometry collision mesh filename=/home/yc/vx300s-single-sim/src/vx300s_description/vx300s_me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 scale=0.001 0.001 0.001; visual mesh filename=/home/yc/vx300s-single-sim/src/vx300s_description/vx300s_me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 scale=0.001 0.001 0.001
- link vx300s/upper_arm_link: geometry collision mesh filename=/home/yc/vx300s-single-sim/src/vx300s_description/vx300s_me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 scale=0.001 0.001 0.001; visual mesh filename=/home/yc/vx300s-single-sim/src/vx300s_description/vx300s_me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 scale=0.001 0.001 0.001
- link vx300s/upper_forearm_link: geometry collision mesh filename=/home/yc/vx300s-single-sim/src/vx300s_description/vx300s_me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 scale=0.001 0.001 0.001; visual mesh filename=/home/yc/vx300s-single-sim/src/vx300s_description/vx300s_me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 scale=0.001 0.001 0.001
- link vx300s/wrist_link: geometry collision mesh filename=/home/yc/vx300s-single-sim/src/vx300s_description/vx300s_me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 scale=0.001 0.001 0.001; visual mesh filename=/home/yc/vx300s-single-sim/src/vx300s_description/vx300s_me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 scale=0.001 0.001 0.001
