Commit message: finish gazebo building, then start to wrtite the computeTorque control method

File: src/vx300s_description/urdf/ros2_control.urdf.xacro (robot description, xacro)
@@ -1,111 +1,165 @@
 <?xml version="1.0"?>
 <robot xmlns:xacro="http://ros.org/wiki/xacro">
-  <ros2_control name="XSHardwareInterface" type="system">
+<xacro:macro name="vx300s_ros2_control">
+  <ros2_control name="vx300sHardwareSystem" type="system">
     <hardware>
-      <!-- If we are using the actual, physical robot -->
-      <xacro:if value="${hardware_type == 'actual'}">
-        <plugin>interbotix_xs_ros_control/XSHardwareInterface</plugin>
-        <param name="loop_hz">10</param>
-        <param name="group_name">arm</param>
-        <param name="gripper_name">gripper</param>
-        <param name="joint_states_topic">joint_states</param>
-      </xacro:if>
-      <!-- If doing basic simulation of the robot -->
-      <xacro:if value="${hardware_type == 'fake'}">
-        <plugin>fake_components/GenericSystem</plugin>
-      </xacro:if>
-      <!-- If simulating the robot in Gazebo Classic -->
-      <xacro:if value="${hardware_type == 'gz_classic'}">
         <plugin>gazebo_ros2_control/GazeboSystem</plugin>
-      </xacro:if>
     </hardware>
+    <!-- Waist -->
     <joint name="waist">
       <command_interface name="position">
-        <param name="min">"${waist_limit_lower}"</param>
-        <param name="max">"${waist_limit_upper}"</param>
+        <param name="min">-3.1416</param>
+        <param name="max">3.1416</param>
+      </command_interface>
+      <command_interface name="velocity">
+        <param name="min">0</param>
+        <param name="max">3.1416</param>
+      </command_interface>
+      <command_interface name="effort">
+        <param name="min">0</param>
+        <param name="max">10</param>
       </command_interface>
       <state_interface name="position"/>
+      <state_interface name="velocity"/>
+      <state_interface name="effort"/>
     </joint>
+    <!-- Shoulder -->
     <joint name="shoulder">
       <command_interface name="position">
-        <param name="min">"${shoulder_limit_lower}"</param>
-        <param name="max">"${shoulder_limit_upper}"</param>
+        <param name="min">-1.8500</param>
+        <param name="max">1.2566</param>
+      </command_interface>
+      <command_interface name="velocity">
+        <param name="min">0</param>
+        <param name="max">3.1416</param>
+      </command_interface>
+      <command_interface name="effort">
+        <param name="min">0</param>
+        <param name="max">20</param>
       </command_interface>
       <state_interface name="position"/>
+      <state_interface name="velocity"/>
+      <state_interface name="effort"/>
     </joint>
+    <!-- Elbow -->
     <joint name="elbow">
       <command_interface name="position">
-        <param name="min">"${elbow_limit_lower}"</param>
-        <param name="max">"${elbow_limit_upper}"</param>
+        <param name="min">-1.7628</param>
+        <param name="max">1.6057</param>
+      </command_interface>
+      <command_interface name="velocity">
+        <param name="min">0</param>
+        <param name="max">3.1416</param>
+      </command_interface>
+      <command_interface name="effort">
+        <param name="min">0</param>
+        <param name="max">15</param>
       </command_interface>
       <state_interface name="position"/>
+      <state_interface name="velocity"/>
+      <state_interface name="effort"/>
     </joint>
-    <xacro:if value="${dof >= 6}">
-      <joint name="forearm_roll">
-        <command_interface name="position">
-          <param name="min">"${forearm_roll_limit_lower}"</param>
-          <param name="max">"${forearm_roll_limit_upper}"</param>
-        </command_interface>
-        <state_interface name="position"/>
-      </joint>
-    </xacro:if>
+    <!-- Forearm roll -->
+    <joint name="forearm_roll">
+      <command_interface name="position">
+        <param name="min">-3.1416</param>
+        <param name="max">3.1416</param>
+      </command_interface>
+      <command_interface name="velocity">
+        <param name="min">0</param>
+        <param name="max">3.1416</param>
+      </command_interface>
+      <command_interface name="effort">
+        <param name="min">0</param>
+        <param name="max">2</param>
+      </command_interface>
+      <state_interface name="position"/>
+      <state_interface name="velocity"/>
+      <state_interface name="effort"/>
+    </joint>
+    <!-- Wrist angle -->
     <joint name="wrist_angle">
       <command_interface name="position">
-        <param name="min">"${wrist_angle_limit_lower}"</param>
-        <param name="max">"${wrist_angle_limit_upper}"</param>
+        <param name="min">-1.8675</param>
+        <param name="max">2.2340</param>
+      </command_interface>
+      <command_interface name="velocity">
+        <param name="min">0</param>
+        <param name="max">3.1416</param>
+      </command_interface>
+      <command_interface name="effort">
+        <param name="min">0</param>
+        <param name="max">5</param>
       </command_interface>
       <state_interface name="position"/>
+      <state_interface name="velocity"/>
+      <state_interface name="effort"/>
     </joint>
-    <xacro:if value="${dof >= 5}">
-      <joint name="wrist_rotate">
-        <command_interface name="position">
-          <param name="min">"${wrist_rotate_limit_lower}"</param>
-          <param name="max">"${wrist_rotate_limit_upper}"</param>
-        </command_interface>
-        <state_interface name="position"/>
-      </joint>
-    </xacro:if>
-    <xacro:if value="$(arg use_gripper)">
-      <xacro:if value="${hardware_type in ('fake', 'gz_classic')}">
-        <joint name="gripper">
-          <command_interface name="position"/>
-          <state_interface name="position"/>
-        </joint>
-      </xacro:if>
-      <xacro:if value="$(arg show_gripper_fingers)">
-        <joint name="left_finger">
-          <command_interface name="position">
-            <param name="min">"${finger_limit_lower}"</param>
-            <param name="max">"${-finger_limit_lower}"</param>
-          </command_interface>
-          <state_interface name="position"/>
-        </joint>
-        <xacro:if value="${hardware_type == 'gz_classic'}">
-          <joint name="right_finger">
-            <!-- <param name="mimic">left_finger</param>
-            <param name="multiplier">1</param> -->
-            <command_interface name="position">
-              <param name="min">"${-finger_limit_lower}"</param>
-              <param name="max">"${finger_limit_lower}"</param>
-            </command_interface>
-            <state_interface name="position"/>
-          </joint>
-        </xacro:if>
-      </xacro:if>
-    </xacro:if>
+    <!-- Wrist rotate -->
+    <joint name="wrist_rotate">
+      <command_interface name="position">
+        <param name="min">-3.1416</param>
+        <param name="max">3.1416</param>
+      </command_interface>
+      <command_interface name="velocity">
+        <param name="min">0</param>
+        <param name="max">3.1416</param>
+      </command_interface>
+      <command_interface name="effort">
+        <param name="min">0</param>
+        <param name="max">1</param>
+      </command_interface>
+      <state_interface name="position"/>
+      <state_interface name="velocity"/>
+      <state_interface name="effort"/>
+    </joint>
+    <!-- Gripper (simple) -->
+    <joint name="gripper">
+      <command_interface name="position"/>
+      <state_interface name="position"/>
+    </joint>
+    <!-- Left finger -->
+    <joint name="left_finger">
+      <command_interface name="position">
+        <param name="min">0.021</param>
+        <param name="max">0.057</param>
+      </command_interface>
+      <command_interface name="velocity">
+        <param name="min">0</param>
+        <param name="max">1.0</param>
+      </command_interface>
+      <command_interface name="effort">
+        <param name="min">0</param>
+        <param name="max">5</param>
+      </command_interface>
+      <state_interface name="position"/>
+      <state_interface name="velocity"/>
+      <state_interface name="effort"/>
+    </joint>
+    <!-- Right finger -->
+    <joint name="right_finger">
+      <command_interface name="position">
+        <param name="min">-0.057</param>
+        <param name="max">-0.021</param>
+      </command_interface>
+      <command_interface name="velocity">
+        <param name="min">0</param>
+        <param name="max">1.0</param>
+      </command_interface>
+      <command_interface name="effort">
+        <param name="min">0</param>
+        <param name="max">5</param>
+      </command_interface>
+      <state_interface name="position"/>
+      <state_interface name="velocity"/>
+      <state_interface name="effort"/>
+    </joint>
   </ros2_control>
-  <!-- Load the gazebo_ros2_control plugin if using Gazebo hardware -->
-  <xacro:if value="${hardware_type == 'gz_classic'}">
-    <gazebo>
-      <plugin filename="libgazebo_ros2_control.so" name="gazebo_ros2_control">
-        <ros>
-          <namespace>/$(arg robot_name)</namespace>
-        </ros>
-        <robot_param>robot_description</robot_param>
-        <robot_param_node>robot_state_publisher</robot_param_node>
-        <parameters>$(find interbotix_xsarm_sim)/config/trajectory_controllers/${robot_model}_trajectory_controllers.yaml</parameters>
-      </plugin>
-    </gazebo>
-    <xacro:include filename="$(find interbotix_common_sim)/media/materials/scripts/interbotix_texture.gazebo"/>
-  </xacro:if>
+  <!-- Gazebo ros2_control plugin -->
+  <gazebo>
+    <plugin filename="libgazebo_ros2_control.so" name="gazebo_ros2_control">
+      <parameters>$(find vx300s_description)/config/vx300s_ros2_controller.yaml</parameters>
+    </plugin>
+  </gazebo>
+</xacro:macro>
 </robot>

File: src/vx300s_description/urdf/vx300s.urdf.xacro (robot description, xacro)
@@ -2,5 +2,5 @@
 <robot xmlns:xacro="http://www.ros.org/wiki/xacro" name="vx300s">
   <material name="interbotix_black">
-    <texture filename="file:///home/yc/vx300s-single-sim/src/vx300s_description/vx300s_meshes/interbotix_black.png"/>
+    <texture filename="$(find vx300s_description)/vx300s_meshes/interbotix_black.png"/>
   </material>
   <!-- use_world_frame -->
@@ -10,5 +10,5 @@
        <origin rpy="0 0 1.5707963267948966" xyz="0 0 0"/>
        <geometry>
-         <mesh filename="file:///home/yc/vx300s-single-sim/src/vx300s_description/vx300s_meshes/base.stl" scale="0.001 0.001 0.001"/>
+         <mesh filename="$(find vx300s_description)/vx300s_meshes/base.stl" scale="0.001 0.001 0.001"/>
        </geometry>
        <material name="interbotix_black"/>
@@ -17,5 +17,5 @@
        <origin rpy="0 0 1.5707963267948966" xyz="0 0 0"/>
        <geometry>
-         <mesh filename="file:///home/yc/vx300s-single-sim/src/vx300s_description/vx300s_meshes/base.stl" scale="0.001 0.001 0.001"/>
+         <mesh filename="$(find vx300s_description)/vx300s_meshes/base.stl" scale="0.001 0.001 0.001"/>
        </geometry>
      </collision>
@@ -38,5 +38,5 @@
       <origin rpy="0 0 1.5707963267948966" xyz="0 0 -0.003"/>
       <geometry>
-        <mesh filename="file:///home/yc/vx300s-single-sim/src/vx300s_description/vx300s_meshes/shoulder.stl" scale="0.001 0.001 0.001"/>
+        <mesh filename="$(find vx300s_description)/vx300s_meshes/shoulder.stl" scale="0.001 0.001 0.001"/>
       </geometry>
       <material name="interbotix_black"/>
@@ -45,5 +45,5 @@
       <origin rpy="0 0 1.5707963267948966" xyz="0 0 -0.003"/>
       <geometry>
-        <mesh filename="file:///home/yc/vx300s-single-sim/src/vx300s_description/vx300s_meshes/shoulder.stl" scale="0.001 0.001 0.001"/>
+        <mesh filename="$(find vx300s_description)/vx300s_meshes/shoulder.stl" scale="0.001 0.001 0.001"/>
       </geometry>
     </collision>
@@ -66,5 +66,5 @@
       <origin rpy="0 0 1.5707963267948966" xyz="0 0 0"/>
       <geometry>
-        <mesh filename="file:///home/yc/vx300s-single-sim/src/vx300s_description/vx300s_meshes/upper_arm.stl" scale="0.001 0.001 0.001"/>
+        <mesh filename="$(find vx300s_description)/vx300s_meshes/upper_arm.stl" scale="0.001 0.001 0.001"/>
       </geometry>
       <material name="interbotix_black"/>
@@ -73,5 +73,5 @@
       <origin rpy="0 0 1.5707963267948966" xyz="0 0 0"/>
       <geometry>
-        <mesh filename="file:///home/yc/vx300s-single-sim/src/vx300s_description/vx300s_meshes/upper_arm.stl" scale="0.001 0.001 0.001"/>
+        <mesh filename="$(find vx300s_description)/vx300s_meshes/upper_arm.stl" scale="0.001 0.001 0.001"/>
       </geometry>
     </collision>
@@ -94,5 +94,5 @@
       <origin rpy="0 0 0" xyz="0 0 0"/>
       <geometry>
-        <mesh filename="file:///home/yc/vx300s-single-sim/src/vx300s_description/vx300s_meshes/upper_forearm.stl" scale="0.001 0.001 0.001"/>
+        <mesh filename="$(find vx300s_description)/vx300s_meshes/upper_forearm.stl" scale="0.001 0.001 0.001"/>
       </geometry>
       <material name="interbotix_black"/>
@@ -101,5 +101,5 @@
       <origin rpy="0 0 0" xyz="0 0 0"/>
       <geometry>
-        <mesh filename="file:///home/yc/vx300s-single-sim/src/vx300s_description/vx300s_meshes/upper_forearm.stl" scale="0.001 0.001 0.001"/>
+        <mesh filename="$(find vx300s_description)/vx300s_meshes/upper_forearm.stl" scale="0.001 0.001 0.001"/>
       </geometry>
     </collision>
@@ -122,5 +122,5 @@
       <origin rpy="3.141592653589793 0 0" xyz="0 0 0"/>
       <geometry>
-        <mesh filename="file:///home/yc/vx300s-single-sim/src/vx300s_description/vx300s_meshes/lower_forearm.stl" scale="0.001 0.001 0.001"/>
+        <mesh filename="$(find vx300s_description)/vx300s_meshes/lower_forearm.stl" scale="0.001 0.001 0.001"/>
       </geometry>
       <material name="interbotix_black"/>
@@ -129,5 +129,5 @@
       <origin rpy="3.141592653589793 0 0" xyz="0 0 0"/>
       <geometry>
-        <mesh filename="file:///home/yc/vx300s-single-sim/src/vx300s_description/vx300s_meshes/lower_forearm.stl" scale="0.001 0.001 0.001"/>
+        <mesh filename="$(find vx300s_description)/vx300s_meshes/lower_forearm.stl" scale="0.001 0.001 0.001"/>
       </geometry>
     </collision>
@@ -150,5 +150,5 @@
       <origin rpy="0 0 1.5707963267948966" xyz="0 0 0"/>
       <geometry>
-        <mesh filename="file:///home/yc/vx300s-single-sim/src/vx300s_description/vx300s_meshes/wrist.stl" scale="0.001 0.001 0.001"/>
+        <mesh filename="$(find vx300s_description)/vx300s_meshes/wrist.stl" scale="0.001 0.001 0.001"/>
       </geometry>
       <material name="interbotix_black"/>
@@ -157,5 +157,5 @@
       <origin rpy="0 0 1.5707963267948966" xyz="0 0 0"/>
       <geometry>
-        <mesh filename="file:///home/yc/vx300s-single-sim/src/vx300s_description/vx300s_meshes/wrist.stl" scale="0.001 0.001 0.001"/>
+        <mesh filename="$(find vx300s_description)/vx300s_meshes/wrist.stl" scale="0.001 0.001 0.001"/>
       </geometry>
     </collision>
@@ -179,5 +179,5 @@
       <origin rpy="0 0 1.5707963267948966" xyz="-0.02 0 0"/>
       <geometry>
-        <mesh filename="file:///home/yc/vx300s-single-sim/src/vx300s_description/vx300s_meshes/gripper.stl" scale="0.001 0.001 0.001"/>
+        <mesh filename="$(find vx300s_description)/vx300s_meshes/gripper.stl" scale="0.001 0.001 0.001"/>
       </geometry>
       <material name="interbotix_black"/>
@@ -186,5 +186,5 @@
       <origin rpy="0 0 1.5707963267948966" xyz="-0.02 0 0"/>
       <geometry>
-        <mesh filename="file:///home/yc/vx300s-single-sim/src/vx300s_description/vx300s_meshes/gripper.stl" scale="0.001 0.001 0.001"/>
+        <mesh filename="$(find vx300s_description)/vx300s_meshes/gripper.stl" scale="0.001 0.001 0.001"/>
       </geometry>
     </collision>
@@ -219,5 +219,5 @@
       <origin rpy="0 0 1.5707963267948966" xyz="-0.0685 0 0"/>
       <geometry>
-        <mesh filename="file:///home/yc/vx300s-single-sim/src/vx300s_description/vx300s_meshes/gripper_prop.stl" scale="0.001 0.001 0.001"/>
+        <mesh filename="$(find vx300s_description)/vx300s_meshes/gripper_prop.stl" scale="0.001 0.001 0.001"/>
       </geometry>
       <material name="interbotix_black"/>
@@ -226,5 +226,5 @@
       <origin rpy="0 0 1.5707963267948966" xyz="-0.0685 0 0"/>
       <geometry>
-        <mesh filename="file:///home/yc/vx300s-single-sim/src/vx300s_description/vx300s_meshes/gripper_prop.stl" scale="0.001 0.001 0.001"/>
+        <mesh filename="$(find vx300s_description)/vx300s_meshes/gripper_prop.stl" scale="0.001 0.001 0.001"/>
       </geometry>
     </collision>
@@ -242,5 +242,5 @@
       <origin rpy="0 0 1.5707963267948966" xyz="-0.063 0 0"/>
       <geometry>
-        <mesh filename="file:///home/yc/vx300s-single-sim/src/vx300s_description/vx300s_meshes/gripper_bar.stl" scale="0.001 0.001 0.001"/>
+        <mesh filename="$(find vx300s_description)/vx300s_meshes/gripper_bar.stl" scale="0.001 0.001 0.001"/>
       </geometry>
       <material name="interbotix_black"/>
@@ -249,5 +249,5 @@
       <origin rpy="0 0 1.5707963267948966" xyz="-0.063 0 0"/>
       <geometry>
-        <mesh filename="file:///home/yc/vx300s-single-sim/src/vx300s_description/vx300s_meshes/gripper_bar.stl" scale="0.001 0.001 0.001"/>
+        <mesh filename="$(find vx300s_description)/vx300s_meshes/gripper_bar.stl" scale="0.001 0.001 0.001"/>
       </geometry>
     </collision>
@@ -280,5 +280,5 @@
       <origin rpy="1.5707963267948966 -3.141592653589793 1.5707963267948966" xyz="-0.0404 -0.0575 0"/>
       <geometry>
-        <mesh filename="file:///home/yc/vx300s-single-sim/src/vx300s_description/vx300s_meshes/gripper_finger.stl" scale="0.001 0.001 0.001"/>
+        <mesh filename="$(find vx300s_description)/vx300s_meshes/gripper_finger.stl" scale="0.001 0.001 0.001"/>
       </geometry>
       <material name="interbotix_black"/>
@@ -287,5 +287,5 @@
       <origin rpy="1.5707963267948966 -3.141592653589793 1.5707963267948966" xyz="-0.0404 -0.0575 0"/>
       <geometry>
-        <mesh filename="file:///home/yc/vx300s-single-sim/src/vx300s_description/vx300s_meshes/gripper_finger.stl" scale="0.001 0.001 0.001"/>
+        <mesh filename="$(find vx300s_description)/vx300s_meshes/gripper_finger.stl" scale="0.001 0.001 0.001"/>
       </geometry>
     </collision>
@@ -317,5 +317,5 @@
       <origin rpy="-1.5707963267948966 3.141592653589793 -1.5707963267948966" xyz="-0.0404 0.0575 0 "/>
       <geometry>
-        <mesh filename="file:///home/yc/vx300s-single-sim/src/vx300s_description/vx300s_meshes/gripper_finger.stl" scale="0.001 0.001 0.001"/>
+        <mesh filename="$(find vx300s_description)/vx300s_meshes/gripper_finger.stl" scale="0.001 0.001 0.001"/>
       </geometry>
       <material name="interbotix_black"/>
@@ -324,5 +324,5 @@
       <origin rpy="-1.5707963267948966 3.141592653589793 -1.5707963267948966" xyz="-0.0404 0.0575 0 "/>
       <geometry>
-        <mesh filename="file:///home/yc/vx300s-single-sim/src/vx300s_description/vx300s_meshes/gripper_finger.stl" scale="0.001 0.001 0.001"/>
+        <mesh filename="$(find vx300s_description)/vx300s_meshes/gripper_finger.stl" scale="0.001 0.001 0.001"/>
       </geometry>
     </collision>
@@ -346,4 +346,6 @@
   </link>
 </xacro:macro>
-    <xacro:vx300s/>
+<xacro:include filename="$(find vx300s_description)/urdf/ros2_control.urdf.xacro"/>
+<xacro:vx300s/>
+<xacro:vx300s_ros2_control/>
 </robot>
