Commit message: GC works

File: src/vx300s_description/urdf/ros2_control.urdf.xacro (robot description, xacro)
@@ -8,14 +8,6 @@
     <!-- Waist -->
     <joint name="waist">
-      <command_interface name="position">
-        <param name="min">-3.1416</param>
-        <param name="max">3.1416</param>
-      </command_interface>
-      <command_interface name="velocity">
-        <param name="min">0</param>
-        <param name="max">3.1416</param>
-      </command_interface>
       <command_interface name="effort">
-        <param name="min">0</param>
+        <param name="min">-10</param>
         <param name="max">10</param>
       </command_interface>
@@ -26,14 +18,6 @@
     <!-- Shoulder -->
     <joint name="shoulder">
-      <command_interface name="position">
-        <param name="min">-1.8500</param>
-        <param name="max">1.2566</param>
-      </command_interface>
-      <command_interface name="velocity">
-        <param name="min">0</param>
-        <param name="max">3.1416</param>
-      </command_interface>
       <command_interface name="effort">
-        <param name="min">0</param>
+        <param name="min">-20</param>
         <param name="max">20</param>
       </command_interface>
@@ -44,14 +28,6 @@
     <!-- Elbow -->
     <joint name="elbow">
-      <command_interface name="position">
-        <param name="min">-1.7628</param>
-        <param name="max">1.6057</param>
-      </command_interface>
-      <command_interface name="velocity">
-        <param name="min">0</param>
-        <param name="max">3.1416</param>
-      </command_interface>
       <command_interface name="effort">
-        <param name="min">0</param>
+        <param name="min">-15</param>
         <param name="max">15</param>
       </command_interface>
@@ -62,14 +38,6 @@
     <!-- Forearm roll -->
     <joint name="forearm_roll">
-      <command_interface name="position">
-        <param name="min">-3.1416</param>
-        <param name="max">3.1416</param>
-      </command_interface>
-      <command_interface name="velocity">
-        <param name="min">0</param>
-        <param name="max">3.1416</param>
-      </command_interface>
       <command_interface name="effort">
-        <param name="min">0</param>
+        <param name="min">-2</param>
         <param name="max">2</param>
       </command_interface>
@@ -80,14 +48,6 @@
     <!-- Wrist angle -->
     <joint name="wrist_angle">
-      <command_interface name="position">
-        <param name="min">-1.8675</param>
-        <param name="max">2.2340</param>
-      </command_interface>
-      <command_interface name="velocity">
-        <param name="min">0</param>
-        <param name="max">3.1416</param>
-      </command_interface>
       <command_interface name="effort">
-        <param name="min">0</param>
+        <param name="min">-5</param>
         <param name="max">5</param>
       </command_interface>
@@ -98,14 +58,6 @@
     <!-- Wrist rotate -->
     <joint name="wrist_rotate">
-      <command_interface name="position">
-        <param name="min">-3.1416</param>
-        <param name="max">3.1416</param>
-      </command_interface>
-      <command_interface name="velocity">
-        <param name="min">0</param>
-        <param name="max">3.1416</param>
-      </command_interface>
       <command_interface name="effort">
-        <param name="min">0</param>
+        <param name="min">-1</param>
         <param name="max">1</param>
       </command_interface>
@@ -118,4 +70,6 @@
       <command_interface name="position"/>
       <state_interface name="position"/>
+      <state_interface name="velocity"/>
+      <state_interface name="effort"/>
     </joint>
     <!-- Left finger -->
@@ -130,5 +84,5 @@
       </command_interface>
       <command_interface name="effort">
-        <param name="min">0</param>
+        <param name="min">-5</param>
         <param name="max">5</param>
       </command_interface>
@@ -148,5 +102,5 @@
       </command_interface>
       <command_interface name="effort">
-        <param name="min">0</param>
+        <param name="min">-5</param>
         <param name="max">5</param>
       </command_interface>

File: src/vx300s_description/urdf/vx300s_fix.urdf (robot description, URDF)
Before this commit: robot vx300s, 15 links, 14 joints
Joints:
- joint gripper: type continuous -> fixed
- joint left_finger: type prismatic -> fixed
- joint right_finger: type prismatic -> fixed

File: src/vx300s_description/urdf/vx300s_fix.urdf.xacro (robot description, xacro)
@@ -1,12 +1,10 @@
 <?xml version="1.0" encoding="utf-8"?>
-<!-- =================================================================================== -->
-<!-- |    This document was autogenerated by xacro from /home/haibo/interbotix_ws/src/interbotix_ros_manipulators/interbotix_ros_xsarms/interbotix_xsarm_descriptions/urdf/vx300s.urdf.xacro | -->
-<!-- |    EDITING THIS FILE BY HAND IS NOT RECOMMENDED                                 | -->
-<!-- =================================================================================== -->
-<robot name="vx300s">
+<robot xmlns:xacro="http://www.ros.org/wiki/xacro" name="vx300s">
   <material name="interbotix_black">
-    <texture filename="/home/haibo/vx300s_ws/src/vx300s_description/vx300s_meshes/interbotix_black.png"/>
+    <texture filename="$(find vx300s_description)/vx300s_meshes/interbotix_black.png"/>
   </material>
-  <link name="world"/>
+  <!-- use_world_frame -->
+<xacro:macro name="vx300s">
+<link name="world"/>
     <joint name="fixed" type="fixed">
       <parent
@@ -15,26 +13,25 @@
         link="vx300s/base_link"/>
     </joint>
-  <!-- use_world_frame -->
-  <link name="vx300s/base_link">
-    <visual>
-      <origin rpy="0 0 1.5707963267948966" xyz="0 0 0"/>
-      <geometry>
-        <mesh filename="/home/haibo/vx300s_ws/src/vx300s_description/vx300s_meshes/base.stl" scale="0.001 0.001 0.001"/>
-      </geometry>
-      <material name="interbotix_black"/>
-    </visual>
-    <collision>
-      <origin rpy="0 0 1.5707963267948966" xyz="0 0 0"/>
-      <geometry>
-        <mesh filename="/home/haibo/vx300s_ws/src/vx300s_description/vx300s_meshes/base.stl" scale="0.001 0.001 0.001"/>
-      </geometry>
-    </collision>
-    <inertial>
-      <origin rpy="0 0 1.5707963267948966" xyz="-0.0534774000 -0.0005625750 0.0205961000"/>
-      <mass value="0.969034"/>
-      <inertia ixx="0.0060240000" ixy="0.0000471300" ixz="0.0000038510" iyy="0.0017000000" iyz="-0.0000841500" izz="0.0071620000"/>
-    </inertial>
-  </link>
-  <joint name="waist" type="revolute">
+ <link name="vx300s/base_link">
+     <visual>
+       <origin rpy="0 0 1.5707963267948966" xyz="0 0 0"/>
+       <geometry>
+         <mesh filename="$(find vx300s_description)/vx300s_meshes/base.stl" scale="0.001 0.001 0.001"/>
+       </geometry>
+       <material name="interbotix_black"/>
+     </visual>
+     <collision>
+       <origin rpy="0 0 1.5707963267948966" xyz="0 0 0"/>
+       <geometry>
+         <mesh filename="$(find vx300s_description)/vx300s_meshes/base.stl" scale="0.001 0.001 0.001"/>
+       </geometry>
+     </collision>
+     <inertial>
+       <origin rpy="0 0 1.5707963267948966" xyz="-0.0534774000 -0.0005625750 0.0205961000"/>
+       <mass value="0.969034"/>
+       <inertia ixx="0.0060240000" ixy="0.0000471300" ixz="0.0000038510" iyy="0.0017000000" iyz="-0.0000841500" izz="0.0071620000"/>
+     </inertial>
+ </link>
+ <joint name="waist" type="revolute">
     <axis xyz="0 0 1"/>
     <limit effort="10" lower="-3.141582653589793" upper="3.141582653589793" velocity="3.141592653589793"/>
@@ -43,10 +40,10 @@
     <child link="vx300s/shoulder_link"/>
     <dynamics damping="0.1" friction="0.1"/>
-  </joint>
+ </joint>
   <link name="vx300s/shoulder_link">
     <visual>
       <origin rpy="0 0 1.5707963267948966" xyz="0 0 -0.003"/>
       <geometry>
-        <mesh filename="/home/haibo/vx300s_ws/src/vx300s_description/vx300s_meshes/shoulder.stl" scale="0.001 0.001 0.001"/>
+        <mesh filename="$(find vx300s_description)/vx300s_meshes/shoulder.stl" scale="0.001 0.001 0.001"/>
       </geometry>
       <material name="interbotix_black"/>
@@ -55,5 +52,5 @@
       <origin rpy="0 0 1.5707963267948966" xyz="0 0 -0.003"/>
       <geometry>
-        <mesh filename="/home/haibo/vx300s_ws/src/vx300s_description/vx300s_meshes/shoulder.stl" scale="0.001 0.001 0.001"/>
+        <mesh filename="$(find vx300s_description)/vx300s_meshes/shoulder.stl" scale="0.001 0.001 0.001"/>
       </geometry>
     </collision>
@@ -76,5 +73,5 @@
       <origin rpy="0 0 1.5707963267948966" xyz="0 0 0"/>
       <geometry>
-        <mesh filename="/home/haibo/vx300s_ws/src/vx300s_description/vx300s_meshes/upper_arm.stl" scale="0.001 0.001 0.001"/>
+        <mesh filename="$(find vx300s_description)/vx300s_meshes/upper_arm.stl" scale="0.001 0.001 0.001"/>
       </geometry>
       <material name="interbotix_black"/>
@@ -83,5 +80,5 @@
       <origin rpy="0 0 1.5707963267948966" xyz="0 0 0"/>
       <geometry>
-        <mesh filename="/home/haibo/vx300s_ws/src/vx300s_description/vx300s_meshes/upper_arm.stl" scale="0.001 0.001 0.001"/>
+        <mesh filename="$(find vx300s_description)/vx300s_meshes/upper_arm.stl" scale="0.001 0.001 0.001"/>
       </geometry>
     </collision>
@@ -104,5 +101,5 @@
       <origin rpy="0 0 0" xyz="0 0 0"/>
       <geometry>
-        <mesh filename="/home/haibo/vx300s_ws/src/vx300s_description/vx300s_meshes/upper_forearm.stl" scale="0.001 0.001 0.001"/>
+        <mesh filename="$(find vx300s_description)/vx300s_meshes/upper_forearm.stl" scale="0.001 0.001 0.001"/>
       </geometry>
       <material name="interbotix_black"/>
@@ -111,5 +108,5 @@
       <origin rpy="0 0 0" xyz="0 0 0"/>
       <geometry>
-        <mesh filename="/home/haibo/vx300s_ws/src/vx300s_description/vx300s_meshes/upper_forearm.stl" scale="0.001 0.001 0.001"/>
+        <mesh filename="$(find vx300s_description)/vx300s_meshes/upper_forearm.stl" scale="0.001 0.001 0.001"/>
       </geometry>
     </collision>
@@ -132,5 +129,5 @@
       <origin rpy="3.141592653589793 0 0" xyz="0 0 0"/>
       <geometry>
-        <mesh filename="/home/haibo/vx300s_ws/src/vx300s_description/vx300s_meshes/lower_forearm.stl" scale="0.001 0.001 0.001"/>
+        <mesh filename="$(find vx300s_description)/vx300s_meshes/lower_forearm.stl" scale="0.001 0.001 0.001"/>
       </geometry>
       <material name="interbotix_black"/>
@@ -139,5 +136,5 @@
       <origin rpy="3.141592653589793 0 0" xyz="0 0 0"/>
       <geometry>
-        <mesh filename="/home/haibo/vx300s_ws/src/vx300s_description/vx300s_meshes/lower_forearm.stl" scale="0.001 0.001 0.001"/>
+        <mesh filename="$(find vx300s_description)/vx300s_meshes/lower_forearm.stl" scale="0.001 0.001 0.001"/>
       </geometry>
     </collision>
@@ -160,5 +157,5 @@
       <origin rpy="0 0 1.5707963267948966" xyz="0 0 0"/>
       <geometry>
-        <mesh filename="/home/haibo/vx300s_ws/src/vx300s_description/vx300s_meshes/wrist.stl" scale="0.001 0.001 0.001"/>
+        <mesh filename="$(find vx300s_description)/vx300s_meshes/wrist.stl" scale="0.001 0.001 0.001"/>
       </geometry>
       <material name="interbotix_black"/>
@@ -167,5 +164,5 @@
       <origin rpy="0 0 1.5707963267948966" xyz="0 0 0"/>
       <geometry>
-        <mesh filename="/home/haibo/vx300s_ws/src/vx300s_description/vx300s_meshes/wrist.stl" scale="0.001 0.001 0.001"/>
+        <mesh filename="$(find vx300s_description)/vx300s_meshes/wrist.stl" scale="0.001 0.001 0.001"/>
       </geometry>
     </collision>
@@ -189,5 +186,5 @@
       <origin rpy="0 0 1.5707963267948966" xyz="-0.02 0 0"/>
       <geometry>
-        <mesh filename="/home/haibo/vx300s_ws/src/vx300s_description/vx300s_meshes/gripper.stl" scale="0.001 0.001 0.001"/>
+        <mesh filename="$(find vx300s_description)/vx300s_meshes/gripper.stl" scale="0.001 0.001 0.001"/>
       </geometry>
       <material name="interbotix_black"/>
@@ -196,5 +193,5 @@
       <origin rpy="0 0 1.5707963267948966" xyz="-0.02 0 0"/>
       <geometry>
-        <mesh filename="/home/haibo/vx300s_ws/src/vx300s_description/vx300s_meshes/gripper.stl" scale="0.001 0.001 0.001"/>
+        <mesh filename="$(find vx300s_description)/vx300s_meshes/gripper.stl" scale="0.001 0.001 0.001"/>
       </geometry>
     </collision>
@@ -217,5 +214,5 @@
     </inertial>
   </link>
-  <joint name="gripper" type="continuous">
+  <joint name="gripper" type="fixed">
     <axis xyz="1 0 0"/>
     <limit effort="1" velocity="3.141592653589793"/>
@@ -225,9 +222,9 @@
     <dynamics damping="0.1" friction="0.1"/>
   </joint>
-  <link name="vx300s/gripper_prop_link">
+ <link name="vx300s/gripper_prop_link">
     <visual>
       <origin rpy="0 0 1.5707963267948966" xyz="-0.0685 0 0"/>
       <geometry>
-        <mesh filename="/home/haibo/vx300s_ws/src/vx300s_description/vx300s_meshes/gripper_prop.stl" scale="0.001 0.001 0.001"/>
+        <mesh filename="$(find vx300s_description)/vx300s_meshes/gripper_prop.stl" scale="0.001 0.001 0.001"/>
       </geometry>
       <material name="interbotix_black"/>
@@ -236,5 +233,5 @@
       <origin rpy="0 0 1.5707963267948966" xyz="-0.0685 0 0"/>
       <geometry>
-        <mesh filename="/home/haibo/vx300s_ws/src/vx300s_description/vx300s_meshes/gripper_prop.stl" scale="0.001 0.001 0.001"/>
+        <mesh filename="$(find vx300s_description)/vx300s_meshes/gripper_prop.stl" scale="0.001 0.001 0.001"/>
       </geometry>
     </collision>
@@ -248,4 +245,24 @@
   <!-- show_ar_tag -->
   <!-- If the gripper bar is being used, then also add the gripper bar -->
+  <link name="vx300s/gripper_bar_link">
+    <visual>
+      <origin rpy="0 0 1.5707963267948966" xyz="-0.063 0 0"/>
+      <geometry>
+        <mesh filename="$(find vx300s_description)/vx300s_meshes/gripper_bar.stl" scale="0.001 0.001 0.001"/>
+      </geometry>
+      <material name="interbotix_black"/>
+    </visual>
+    <collision>
+      <origin rpy="0 0 1.5707963267948966" xyz="-0.063 0 0"/>
+      <geometry>
+        <mesh filename="$(find vx300s_description)/vx300s_meshes/gripper_bar.stl" scale="0.001 0.001 0.001"/>
+      </geometry>
+    </collision>
+    <inertial>
+      <origin rpy="0 0 1.5707963267948966" xyz="0.0067940000 -0.0000004272 -0.0007760000"/>
+      <mass value="0.150986"/>
+      <inertia ixx="0.0000789500" ixy="-0.0000000012" ixz="0.0000001341" iyy="0.0003283000" iyz="0.0000017465" izz="0.0003095000"/>
+    </inertial>
+  </link>
   <joint name="gripper_bar" type="fixed">
     <axis xyz="1 0 0"/>
@@ -254,25 +271,5 @@
     <child link="vx300s/gripper_bar_link"/>
   </joint>
-  <link name="vx300s/gripper_bar_link">
-    <visual>
-      <origin rpy="0 0 1.5707963267948966" xyz="-0.063 0 0"/>
-      <geometry>
-        <mesh filename="/home/haibo/vx300s_ws/src/vx300s_description/vx300s_meshes/gripper_bar.stl" scale="0.001 0.001 0.001"/>
-      </geometry>
-      <material name="interbotix_black"/>
-    </visual>
-    <collision>
-      <origin rpy="0 0 1.5707963267948966" xyz="-0.063 0 0"/>
-      <geometry>
-        <mesh filename="/home/haibo/vx300s_ws/src/vx300s_description/vx300s_meshes/gripper_bar.stl" scale="0.001 0.001 0.001"/>
-      </geometry>
-    </collision>
-    <inertial>
-      <origin rpy="0 0 1.5707963267948966" xyz="0.0067940000 -0.0000004272 -0.0007760000"/>
-      <mass value="0.150986"/>
-      <inertia ixx="0.0000789500" ixy="-0.0000000012" ixz="0.0000001341" iyy="0.0003283000" iyz="0.0000017465" izz="0.0003095000"/>
-    </inertial>
-  </link>
-  <joint name="ee_bar" type="fixed">
+<joint name="ee_bar" type="fixed">
     <axis xyz="1 0 0"/>
     <origin rpy="0 0 0" xyz="0.025875 0 0"/>
@@ -286,6 +283,25 @@
     </inertial>
   </link>
-  <!-- If the gripper fingers are being used, add those as well -->
-  <joint name="left_finger" type="prismatic">
+  <link name="vx300s/left_finger_link">
+    <visual>
+      <origin rpy="1.5707963267948966 -3.141592653589793 1.5707963267948966" xyz="-0.0404 -0.0575 0"/>
+      <geometry>
+        <mesh filename="$(find vx300s_description)/vx300s_meshes/gripper_finger.stl" scale="0.001 0.001 0.001"/>
+      </geometry>
+      <material name="interbotix_black"/>
+    </visual>
+    <collision>
+      <origin rpy="1.5707963267948966 -3.141592653589793 1.5707963267948966" xyz="-0.0404 -0.0575 0"/>
+      <geometry>
+        <mesh filename="$(find vx300s_description)/vx300s_meshes/gripper_finger.stl" scale="0.001 0.001 0.001"/>
+      </geometry>
+    </collision>
+    <inertial>
+      <origin rpy="3.141592653589793 3.141592653589793 1.5707963267948966" xyz="0.0173440000 -0.0060692000 0.0000000000"/>
+      <mass value="0.034796"/>
+      <inertia ixx="0.0000243300" ixy="-0.0000024004" ixz="0.0000000000" iyy="0.0000125500" iyz="0.0000000000" izz="0.0000141700"/>
+    </inertial>
+  </link>
+<joint name="left_finger" type="fixed">
     <axis xyz="0 1 0"/>
     <limit effort="5" lower="0.021" upper="0.057" velocity="1"/>
@@ -295,25 +311,5 @@
     <dynamics damping="0.1" friction="0.1"/>
   </joint>
-  <link name="vx300s/left_finger_link">
-    <visual>
-      <origin rpy="1.5707963267948966 -3.141592653589793 1.5707963267948966" xyz="-0.0404 -0.0575 0"/>
-      <geometry>
-        <mesh filename="/home/haibo/vx300s_ws/src/vx300s_description/vx300s_meshes/gripper_finger.stl" scale="0.001 0.001 0.001"/>
-      </geometry>
-      <material name="interbotix_black"/>
-    </visual>
-    <collision>
-      <origin rpy="1.5707963267948966 -3.141592653589793 1.5707963267948966" xyz="-0.0404 -0.0575 0"/>
-      <geometry>
-        <mesh filename="/home/haibo/vx300s_ws/src/vx300s_description/vx300s_meshes/gripper_finger.stl" scale="0.001 0.001 0.001"/>
-      </geometry>
-    </collision>
-    <inertial>
-      <origin rpy="3.141592653589793 3.141592653589793 1.5707963267948966" xyz="0.0173440000 -0.0060692000 0.0000000000"/>
-      <mass value="0.034796"/>
-      <inertia ixx="0.0000243300" ixy="-0.0000024004" ixz="0.0000000000" iyy="0.0000125500" iyz="0.0000000000" izz="0.0000141700"/>
-    </inertial>
-  </link>
-  <joint name="right_finger" type="prismatic">
+<joint name="right_finger" type="fixed">
     <axis xyz="0 1 0"/>
     <limit effort="5" lower="-0.057" upper="-0.021" velocity="1"/>
@@ -328,5 +324,5 @@
       <origin rpy="-1.5707963267948966 3.141592653589793 -1.5707963267948966" xyz="-0.0404 0.0575 0 "/>
       <geometry>
-        <mesh filename="/home/haibo/vx300s_ws/src/vx300s_description/vx300s_meshes/gripper_finger.stl" scale="0.001 0.001 0.001"/>
+        <mesh filename="$(find vx300s_description)/vx300s_meshes/gripper_finger.stl" scale="0.001 0.001 0.001"/>
       </geometry>
       <material name="interbotix_black"/>
@@ -335,5 +331,5 @@
       <origin rpy="-1.5707963267948966 3.141592653589793 -1.5707963267948966" xyz="-0.0404 0.0575 0 "/>
       <geometry>
-        <mesh filename="/home/haibo/vx300s_ws/src/vx300s_description/vx300s_meshes/gripper_finger.stl" scale="0.001 0.001 0.001"/>
+        <mesh filename="$(find vx300s_description)/vx300s_meshes/gripper_finger.stl" scale="0.001 0.001 0.001"/>
       </geometry>
     </collision>
@@ -344,5 +340,5 @@
     </inertial>
   </link>
-  <joint name="ee_gripper" type="fixed">
+<joint name="ee_gripper" type="fixed">
     <axis xyz="1 0 0"/>
     <origin rpy="0 0 0" xyz="0.0385 0 0"/>
@@ -356,6 +352,7 @@
     </inertial>
   </link>
-  <!-- show_gripper_fingers -->
-  <!-- show_gripper_bar -->
-  <!-- use_gripper -->
+</xacro:macro>
+<xacro:include filename="$(find vx300s_description)/urdf/ros2_control.urdf.xacro"/>
+<xacro:vx300s/>
+<xacro:vx300s_ros2_control/>
 </robot>
