Commit message: fianl version

File: src/vx300s_description/urdf/ros2_control.urdf.xacro (robot description, xacro)
@@ -9,5 +9,5 @@
     <joint name="waist">
       <command_interface name="effort">
-        <param name="min">-10</param>
+        <param name="min">0</param>
         <param name="max">10</param>
       </command_interface>
@@ -19,5 +19,5 @@
     <joint name="shoulder">
       <command_interface name="effort">
-        <param name="min">-20</param>
+        <param name="min">0</param>
         <param name="max">20</param>
       </command_interface>
@@ -29,5 +29,5 @@
     <joint name="elbow">
       <command_interface name="effort">
-        <param name="min">-15</param>
+        <param name="min">0</param>
         <param name="max">15</param>
       </command_interface>
@@ -39,5 +39,5 @@
     <joint name="forearm_roll">
       <command_interface name="effort">
-        <param name="min">-2</param>
+        <param name="min">0</param>
         <param name="max">2</param>
       </command_interface>
@@ -49,5 +49,5 @@
     <joint name="wrist_angle">
       <command_interface name="effort">
-        <param name="min">-5</param>
+        <param name="min">0</param>
         <param name="max">5</param>
       </command_interface>
@@ -59,5 +59,5 @@
     <joint name="wrist_rotate">
       <command_interface name="effort">
-        <param name="min">-1</param>
+        <param name="min">0</param>
         <param name="max">1</param>
       </command_interface>
@@ -84,5 +84,5 @@
       </command_interface>
       <command_interface name="effort">
-        <param name="min">-5</param>
+        <param name="min">0</param>
         <param name="max">5</param>
       </command_interface>
@@ -94,5 +94,5 @@
     <joint name="right_finger">
       <command_interface name="position">
-        <param name="min">-0.057</param>
+        <param name="min">0</param>
         <param name="max">-0.021</param>
       </command_interface>
@@ -102,5 +102,5 @@
       </command_interface>
       <command_interface name="effort">
-        <param name="min">-5</param>
+        <param name="min">0</param>
         <param name="max">5</param>
       </command_interface>

File: src/vx300s_description/urdf/vx300s.urdf (robot description, URDF)
Before this commit: robot vx300s, 15 links, 14 joints
Links:
- link vx300s/base_link: geometry collision mesh filename=/home/yc/vx300s-single-sim/src/vx300s_description/vx300s_me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 scale=0.001 0.001 0.001; visual mesh filename=/home/yc/vx300s-single-sim/src/vx300s_description/vx300s_me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 scale=0.001 0.001 0.001
- link vx300s/gripper_bar_link: geometry collision mesh filename=/home/yc/vx300s-single-sim/src/vx300s_description/vx300s_me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 scale=0.001 0.001 0.001; visual mesh filename=/home/yc/vx300s-single-sim/src/vx300s_description/vx300s_me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 scale=0.001 0.001 0.001
- link vx300s/gripper_link: geometry collision mesh filename=/home/yc/vx300s-single-sim/src/vx300s_description/vx300s_me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 scale=0.001 0.001 0.001; visual mesh filename=/home/yc/vx300s-single-sim/src/vx300s_description/vx300s_me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 scale=0.001 0.001 0.001
- link vx300s/gripper_prop_link: geometry collision mesh filename=/home/yc/vx300s-single-sim/src/vx300s_description/vx300s_me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 scale=0.001 0.001 0.001; visual mesh filename=/home/yc/vx300s-single-sim/src/vx300s_description/vx300s_me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 scale=0.001 0.001 0.001
- link vx300s/left_finger_link: geometry collision mesh filename=/home/yc/vx300s-single-sim/src/vx300s_description/vx300s_me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 scale=0.001 0.001 0.001; visual mesh filename=/home/yc/vx300s-single-sim/src/vx300s_description/vx300s_me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 scale=0.001 0.001 0.001
- link vx300s/lower_forearm_link: geometry collision mesh filename=/home/yc/vx300s-single-sim/src/vx300s_description/vx300s_me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 scale=0.001 0.001 0.001; visual mesh filename=/home/yc/vx300s-single-sim/src/vx300s_description/vx300s_me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 scale=0.001 0.001 0.001
- link vx300s/right_finger_link: geometry collision mesh filename=/home/yc/vx300s-single-sim/src/vx300s_description/vx300s_me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 scale=0.001 0.001 0.001; visual mesh filename=/home/yc/vx300s-single-sim/src/vx300s_description/vx300s_me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 scale=0.001 0.001 0.001
- link vx300s/shoulder_link: geometry collision mesh filename=/home/yc/vx300s-single-sim/src/vx300s_description/vx300s_me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 scale=0.001 0.001 0.001; visual mesh filename=/home/yc/vx300s-single-sim/src/vx300s_description/vx300s_me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 scale=0.001 0.001 0.001
- link vx300s/upper_arm_link: geometry collision mesh filename=/home/yc/vx300s-single-sim/src/vx300s_description/vx300s_me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 scale=0.001 0.001 0.001; visual mesh filename=/home/yc/vx300s-single-sim/src/vx300s_description/vx300s_me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 scale=0.001 0.001 0.001
- link vx300s/upper_forearm_link: geometry collision mesh filename=/home/yc/vx300s-single-sim/src/vx300s_description/vx300s_me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 scale=0.001 0.001 0.001; visual mesh filename=/home/yc/vx300s-single-sim/src/vx300s_description/vx300s_me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 scale=0.001 0.001 0.001
- link vx300s/wrist_link: geometry collision mesh filename=/home/yc/vx300s-single-sim/src/vx300s_description/vx300s_me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 scale=0.001 0.001 0.001; visual mesh filename=/home/yc/vx300s-single-sim/src/vx300s_description/vx300s_me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 scale=0.001 0.001 0.001

File: src/vx300s_description/urdf/vx300s_fix.urdf (robot description, URDF)
Before this commit: robot vx300s, 15 links, 14 joints
Links:
- link vx300s/base_link: geometry collision mesh filename=/home/yc/vx300s-single-sim/src/vx300s_description/vx300s_me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 scale=0.001 0.001 0.001; visual mesh filename=/home/yc/vx300s-single-sim/src/vx300s_description/vx300s_me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 scale=0.001 0.001 0.001
- link vx300s/gripper_bar_link: geometry collision mesh filename=/home/yc/vx300s-single-sim/src/vx300s_description/vx300s_me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 scale=0.001 0.001 0.001; visual mesh filename=/home/yc/vx300s-single-sim/src/vx300s_description/vx300s_me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 scale=0.001 0.001 0.001
- link vx300s/gripper_link: geometry collision mesh filename=/home/yc/vx300s-single-sim/src/vx300s_description/vx300s_me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 scale=0.001 0.001 0.001; visual mesh filename=/home/yc/vx300s-single-sim/src/vx300s_description/vx300s_me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 scale=0.001 0.001 0.001
- link vx300s/gripper_prop_link: geometry collision mesh filename=/home/yc/vx300s-single-sim/src/vx300s_description/vx300s_me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 scale=0.001 0.001 0.001; visual mesh filename=/home/yc/vx300s-single-sim/src/vx300s_description/vx300s_me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 scale=0.001 0.001 0.001
- link vx300s/left_finger_link: geometry collision mesh filename=/home/yc/vx300s-single-sim/src/vx300s_description/vx300s_me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 scale=0.001 0.001 0.001; visual mesh filename=/home/yc/vx300s-single-sim/src/vx300s_description/vx300s_me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 scale=0.001 0.001 0.001
- link vx300s/lower_forearm_link: geometry collision mesh filename=/home/yc/vx300s-single-sim/src/vx300s_description/vx300s_me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 scale=0.001 0.001 0.001; visual mesh filename=/home/yc/vx300s-single-sim/src/vx300s_description/vx300s_me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 scale=0.001 0.001 0.001
- link vx300s/right_finger_link: geometry collision mesh filename=/home/yc/vx300s-single-sim/src/vx300s_description/vx300s_me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 scale=0.001 0.001 0.001; visual mesh filename=/home/yc/vx300s-single-sim/src/vx300s_description/vx300s_me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 scale=0.001 0.001 0.001
- link vx300s/shoulder_link: geometry collision mesh filename=/home/yc/vx300s-single-sim/src/vx300s_description/vx300s_me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 scale=0.001 0.001 0.001; visual mesh filename=/home/yc/vx300s-single-sim/src/vx300s_description/vx300s_me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 scale=0.001 0.001 0.001
- link vx300s/upper_arm_link: geometry collision mesh filename=/home/yc/vx300s-single-sim/src/vx300s_description/vx300s_me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 scale=0.001 0.001 0.001; visual mesh filename=/home/yc/vx300s-single-sim/src/vx300s_description/vx300s_me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 scale=0.001 0.001 0.001
- link vx300s/upper_forearm_link: geometry collision mesh filename=/home/yc/vx300s-single-sim/src/vx300s_description/vx300s_me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 scale=0.001 0.001 0.001; visual mesh filename=/home/yc/vx300s-single-sim/src/vx300s_description/vx300s_me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 scale=0.001 0.001 0.001
- link vx300s/wrist_link: geometry collision mesh filename=/home/yc/vx300s-single-sim/src/vx300s_description/vx300s_me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 scale=0.001 0.001 0.001; visual mesh filename=/home/yc/vx300s-single-sim/src/vx300s_description/vx300s_me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 scale=0.001 0.001 0.001
