Commit message: moveit reset for robotic arm

File: src/vx300s_description/urdf/vx300s_AbsolutePath.urdf.xacro (robot description, xacro)
@@ -2,9 +2,9 @@
 <robot xmlns:xacro="http://www.ros.org/wiki/xacro" name="vx300s">
   <material name="interbotix_black">
-    <texture filename="file://$(find vx300s_description)/vx300s_meshes/interbotix_black.png"/>
+    <texture filename="/home/haibo/vx300s_ws/src/vx300s_description/vx300s_meshes/interbotix_black.png"/>
   </material>
   <!-- use_world_frame -->
 <xacro:macro name="vx300s">
-<!-- <link name="world"/>
+<link name="world"/>
     <joint name="fixed" type="fixed">
       <parent
@@ -12,10 +12,10 @@
       <child
         link="vx300s/base_link"/>
-    </joint> -->
+    </joint>
  <link name="vx300s/base_link">
      <visual>
        <origin rpy="0 0 1.5707963267948966" xyz="0 0 0"/>
        <geometry>
-         <mesh filename="file://$(find vx300s_description)/vx300s_meshes/base.stl" scale="0.001 0.001 0.001"/>
+         <mesh filename="/home/haibo/vx300s_ws/src/vx300s_description/vx300s_meshes/base.stl" scale="0.001 0.001 0.001"/>
        </geometry>
        <material name="interbotix_black"/>
@@ -24,5 +24,5 @@
        <origin rpy="0 0 1.5707963267948966" xyz="0 0 0"/>
        <geometry>
-         <mesh filename="file://$(find vx300s_description)/vx300s_meshes/base.stl" scale="0.001 0.001 0.001"/>
+         <mesh filename="/home/haibo/vx300s_ws/src/vx300s_description/vx300s_meshes/base.stl" scale="0.001 0.001 0.001"/>
        </geometry>
      </collision>
@@ -45,5 +45,5 @@
       <origin rpy="0 0 1.5707963267948966" xyz="0 0 -0.003"/>
       <geometry>
-        <mesh filename="file://$(find vx300s_description)/vx300s_meshes/shoulder.stl" scale="0.001 0.001 0.001"/>
+        <mesh filename="/home/haibo/vx300s_ws/src/vx300s_description/vx300s_meshes/shoulder.stl" scale="0.001 0.001 0.001"/>
       </geometry>
       <material name="interbotix_black"/>
@@ -52,5 +52,5 @@
       <origin rpy="0 0 1.5707963267948966" xyz="0 0 -0.003"/>
       <geometry>
-        <mesh filename="file://$(find vx300s_description)/vx300s_meshes/shoulder.stl" scale="0.001 0.001 0.001"/>
+        <mesh filename="/home/haibo/vx300s_ws/src/vx300s_description/vx300s_meshes/shoulder.stl" scale="0.001 0.001 0.001"/>
       </geometry>
     </collision>
@@ -73,5 +73,5 @@
       <origin rpy="0 0 1.5707963267948966" xyz="0 0 0"/>
       <geometry>
-        <mesh filename="file://$(find vx300s_description)/vx300s_meshes/upper_arm.stl" scale="0.001 0.001 0.001"/>
+        <mesh filename="/home/haibo/vx300s_ws/src/vx300s_description/vx300s_meshes/upper_arm.stl" scale="0.001 0.001 0.001"/>
       </geometry>
       <material name="interbotix_black"/>
@@ -80,5 +80,5 @@
       <origin rpy="0 0 1.5707963267948966" xyz="0 0 0"/>
       <geometry>
-        <mesh filename="file://$(find vx300s_description)/vx300s_meshes/upper_arm.stl" scale="0.001 0.001 0.001"/>
+        <mesh filename="/home/haibo/vx300s_ws/src/vx300s_description/vx300s_meshes/upper_arm.stl" scale="0.001 0.001 0.001"/>
       </geometry>
     </collision>
@@ -101,5 +101,5 @@
       <origin rpy="0 0 0" xyz="0 0 0"/>
       <geometry>
-        <mesh filename="file://$(find vx300s_description)/vx300s_meshes/upper_forearm.stl" scale="0.001 0.001 0.001"/>
+        <mesh filename="/home/haibo/vx300s_ws/src/vx300s_description/vx300s_meshes/upper_forearm.stl" scale="0.001 0.001 0.001"/>
       </geometry>
       <material name="interbotix_black"/>
@@ -108,5 +108,5 @@
       <origin rpy="0 0 0" xyz="0 0 0"/>
       <geometry>
-        <mesh filename="file://$(find vx300s_description)/vx300s_meshes/upper_forearm.stl" scale="0.001 0.001 0.001"/>
+        <mesh filename="/home/haibo/vx300s_ws/src/vx300s_description/vx300s_meshes/upper_forearm.stl" scale="0.001 0.001 0.001"/>
       </geometry>
     </collision>
@@ -129,5 +129,5 @@
       <origin rpy="3.141592653589793 0 0" xyz="0 0 0"/>
       <geometry>
-        <mesh filename="file://$(find vx300s_description)/vx300s_meshes/lower_forearm.stl" scale="0.001 0.001 0.001"/>
+        <mesh filename="/home/haibo/vx300s_ws/src/vx300s_description/vx300s_meshes/lower_forearm.stl" scale="0.001 0.001 0.001"/>
       </geometry>
       <material name="interbotix_black"/>
@@ -136,5 +136,5 @@
       <origin rpy="3.141592653589793 0 0" xyz="0 0 0"/>
       <geometry>
-        <mesh filename="file://$(find vx300s_description)/vx300s_meshes/lower_forearm.stl" scale="0.001 0.001 0.001"/>
+        <mesh filename="/home/haibo/vx300s_ws/src/vx300s_description/vx300s_meshes/lower_forearm.stl" scale="0.001 0.001 0.001"/>
       </geometry>
     </collision>
@@ -157,5 +157,5 @@
       <origin rpy="0 0 1.5707963267948966" xyz="0 0 0"/>
       <geometry>
-        <mesh filename="file://$(find vx300s_description)/vx300s_meshes/wrist.stl" scale="0.001 0.001 0.001"/>
+        <mesh filename="/home/haibo/vx300s_ws/src/vx300s_description/vx300s_meshes/wrist.stl" scale="0.001 0.001 0.001"/>
       </geometry>
       <material name="interbotix_black"/>
@@ -164,5 +164,5 @@
       <origin rpy="0 0 1.5707963267948966" xyz="0 0 0"/>
       <geometry>
-        <mesh filename="file://$(find vx300s_description)/vx300s_meshes/wrist.stl" scale="0.001 0.001 0.001"/>
+        <mesh filename="/home/haibo/vx300s_ws/src/vx300s_description/vx300s_meshes/wrist.stl" scale="0.001 0.001 0.001"/>
       </geometry>
     </collision>
@@ -186,5 +186,5 @@
       <origin rpy="0 0 1.5707963267948966" xyz="-0.02 0 0"/>
       <geometry>
-        <mesh filename="file://$(find vx300s_description)/vx300s_meshes/gripper.stl" scale="0.001 0.001 0.001"/>
+        <mesh filename="/home/haibo/vx300s_ws/src/vx300s_description/vx300s_meshes/gripper.stl" scale="0.001 0.001 0.001"/>
       </geometry>
       <material name="interbotix_black"/>
@@ -193,5 +193,5 @@
       <origin rpy="0 0 1.5707963267948966" xyz="-0.02 0 0"/>
       <geometry>
-        <mesh filename="file://$(find vx300s_description)/vx300s_meshes/gripper.stl" scale="0.001 0.001 0.001"/>
+        <mesh filename="/home/haibo/vx300s_ws/src/vx300s_description/vx300s_meshes/gripper.stl" scale="0.001 0.001 0.001"/>
       </geometry>
     </collision>
@@ -226,5 +226,5 @@
       <origin rpy="0 0 1.5707963267948966" xyz="-0.0685 0 0"/>
       <geometry>
-        <mesh filename="file://$(find vx300s_description)/vx300s_meshes/gripper_prop.stl" scale="0.001 0.001 0.001"/>
+        <mesh filename="/home/haibo/vx300s_ws/src/vx300s_description/vx300s_meshes/gripper_prop.stl" scale="0.001 0.001 0.001"/>
       </geometry>
       <material name="interbotix_black"/>
@@ -233,5 +233,5 @@
       <origin rpy="0 0 1.5707963267948966" xyz="-0.0685 0 0"/>
       <geometry>
-        <mesh filename="file://$(find vx300s_description)/vx300s_meshes/gripper_prop.stl" scale="0.001 0.001 0.001"/>
+        <mesh filename="/home/haibo/vx300s_ws/src/vx300s_description/vx300s_meshes/gripper_prop.stl" scale="0.001 0.001 0.001"/>
       </geometry>
     </collision>
@@ -249,5 +249,5 @@
       <origin rpy="0 0 1.5707963267948966" xyz="-0.063 0 0"/>
       <geometry>
-        <mesh filename="file://$(find vx300s_description)/vx300s_meshes/gripper_bar.stl" scale="0.001 0.001 0.001"/>
+        <mesh filename="/home/haibo/vx300s_ws/src/vx300s_description/vx300s_meshes/gripper_bar.stl" scale="0.001 0.001 0.001"/>
       </geometry>
       <material name="interbotix_black"/>
@@ -256,5 +256,5 @@
       <origin rpy="0 0 1.5707963267948966" xyz="-0.063 0 0"/>
       <geometry>
-        <mesh filename="file://$(find vx300s_description)/vx300s_meshes/gripper_bar.stl" scale="0.001 0.001 0.001"/>
+        <mesh filename="/home/haibo/vx300s_ws/src/vx300s_description/vx300s_meshes/gripper_bar.stl" scale="0.001 0.001 0.001"/>
       </geometry>
     </collision>
@@ -287,5 +287,5 @@
       <origin rpy="1.5707963267948966 -3.141592653589793 1.5707963267948966" xyz="-0.0404 -0.0575 0"/>
       <geometry>
-        <mesh filename="file://$(find vx300s_description)/vx300s_meshes/gripper_finger.stl" scale="0.001 0.001 0.001"/>
+        <mesh filename="/home/haibo/vx300s_ws/src/vx300s_description/vx300s_meshes/gripper_finger.stl" scale="0.001 0.001 0.001"/>
       </geometry>
       <material name="interbotix_black"/>
@@ -294,5 +294,5 @@
       <origin rpy="1.5707963267948966 -3.141592653589793 1.5707963267948966" xyz="-0.0404 -0.0575 0"/>
       <geometry>
-        <mesh filename="file://$(find vx300s_description)/vx300s_meshes/gripper_finger.stl" scale="0.001 0.001 0.001"/>
+        <mesh filename="/home/haibo/vx300s_ws/src/vx300s_description/vx300s_meshes/gripper_finger.stl" scale="0.001 0.001 0.001"/>
       </geometry>
     </collision>
@@ -324,5 +324,5 @@
       <origin rpy="-1.5707963267948966 3.141592653589793 -1.5707963267948966" xyz="-0.0404 0.0575 0 "/>
       <geometry>
-        <mesh filename="file://$(find vx300s_description)/vx300s_meshes/gripper_finger.stl" scale="0.001 0.001 0.001"/>
+        <mesh filename="/home/haibo/vx300s_ws/src/vx300s_description/vx300s_meshes/gripper_finger.stl" scale="0.001 0.001 0.001"/>
       </geometry>
       <material name="interbotix_black"/>
@@ -331,5 +331,5 @@
       <origin rpy="-1.5707963267948966 3.141592653589793 -1.5707963267948966" xyz="-0.0404 0.0575 0 "/>
       <geometry>
-        <mesh filename="file://$(find vx300s_description)/vx300s_meshes/gripper_finger.stl" scale="0.001 0.001 0.001"/>
+        <mesh filename="/home/haibo/vx300s_ws/src/vx300s_description/vx300s_meshes/gripper_finger.stl" scale="0.001 0.001 0.001"/>
       </geometry>
     </collision>
@@ -353,5 +353,5 @@
   </link>
 </xacro:macro>
-<xacro:include filename="$(find vx300s_description)/urdf/ros2_control.urdf.xacro"/>
+<xacro:include filename="/home/haibo/vx300s_ws/src/vx300s_description/urdf/ros2_control.urdf.xacro"/>
 <xacro:vx300s/>
 <xacro:vx300s_ros2_control/>

File: src/vx300s_description/urdf/vx300s_moveit.urdf.xacro (robot description, xacro)
@@ -6,11 +6,4 @@
   <!-- use_world_frame -->
 <xacro:macro name="vx300s">
-<!-- <link name="world"/>
-    <joint name="fixed" type="fixed">
-      <parent
-        link="world"/>
-      <child
-        link="vx300s/base_link"/>
-    </joint> -->
  <link name="vx300s/base_link">
      <visual>
@@ -353,6 +346,5 @@
   </link>
 </xacro:macro>
-<xacro:include filename="$(find vx300s_description)/urdf/ros2_control.urdf.xacro"/>
+<xacro:include filename="$(find vx300s_description)/urdf/vx300s.ros2_control.xacro"/>
 <xacro:vx300s/>
-<xacro:vx300s_ros2_control/>
 </robot>
